File: hardware/battery_pack/battery_pack.kicad_pcb (KiCad board)
At the start: 4 copper layers, 130 x 110 mm, 282 parts, among them IC301 BQ24618RGER, IC302 BQ7791504, IC401 STM32C092CCT6, J201 USB_C_Receptacle_USB2.0, J202 Conn_01x02_Male, J401 SW_CONN, J501 UART CONN, J502 DB25_Plug_MountingHoles, Q201 SQJ951EP, Q301 SQJ951EP, Q302 STL45P3LLH6, Q303 STL36DN6F7, Q304 MUN5334DW1, Q305 DMG1012T, Q306 DMG1012T, Q307 DMG1012T, Q309 STL36DN6F7, Q310 DMG1012T, Q501 SQJ951EP, U201 BSS84DW, U202 CYPD3177, U203 T2N7002AK, U401 TCAN1164, U402 TLV70033_SOT23-5, U501 T2N7002AK, Y401 ECX_2236B (10pF)

Commit message: Finished routing. Finall review and re-annotation pending.
Parts:
- removed NT319, NT320, NT322, NT325, NT329: NetTie_2, NetTie:NetTie-2_SMD_Pad0.5mm
- removed R209: 5.1k, Resistor_SMD:R_0805_2012Metric_Pad1.20x1.40mm_HandSolder
- removed TP306: ~, TestPoint:TestPoint_Pad_D1.5mm
- added NT1: NetTie_2, NetTie:NetTie-2_SMD_Pad0.5mm, F.Cu at (178.8, 73.1)
- added NT2: NetTie_2, NetTie:NetTie-2_SMD_Pad0.5mm, F.Cu at (173.0, 69.2)
- NT321, NT328: moved to B.Cu
- NT331: moved to F.Cu
- R316, R350: footprint Resistor_SMD:R_1206_3216Metric -> Resistor_SMD:R_2512_6332Metric
- U202: footprint Package_DFN_QFN:QFN-24-1EP_4x4mm_P0.5mm_EP2.75x2.75mm -> Package_DFN_QFN:QFN-24-1EP_4x4mm_P0.5mm_EP2.65x2.65mm
- moved NT321 254.8 mm to (78.5, 54.0), turned to -90 degrees
- moved NT328 250.3 mm to (79.3, 99.2), turned to -90 degrees
- moved TP315 185.3 mm to (163.3, 55.3)
- moved NT318 151.9 mm to (178.8, 72.4)
- moved TP305 93.7 mm to (151.8, 42.2)
- moved NT324 77.2 mm to (165.0, 80.1), turned to 0 degrees
- moved J401 57.0 mm to (139.0, 80.8), turned to 180 degrees
- moved J501 40.3 mm to (153.0, 103.3), turned to 180 degrees
- moved TP325 22.2 mm to (111.6, 100.2)
- moved TP314 16.8 mm to (131.0, 60.0)
- moved NT313 14.8 mm to (125.0, 68.0), turned to 0 degrees
- moved D402 14.8 mm to (161.6, 109.2), turned to -90 degrees
- moved C329 11.3 mm to (172.5, 90.5)
- moved C328 11.2 mm to (168.4, 90.5)
- moved C302 10.9 mm to (157.5, 49.0), turned to 0 degrees
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Connections:
- C321 pad 1: Net-(C320-Pad1) -> Net-(C321-Pad1)
- C328 pad 1: Earth -> Net-(IC302-SRP)
- C329 pad 1: Net-(C329-Pad1) -> Net-(IC302-SRN)
- IC302 pad 24: Net-(IC302-CTRC) -> Net-(IC302-CTRD)
- IC401 pad 2: unconnected-(IC401-PC14-OSCX_IN-Pad2) -> HPI_SDA
- IC401 pad 29: HPI_SCL -> unconnected-(IC401-PA9-Pad29)
- IC401 pad 32: HPI_SDA -> unconnected-(IC401-PA10-Pad32)
- IC401 pad 47: digSTAT1 -> HPI_SCL
- IC401 pad 48: USB_C_GPIO -> digSTAT1
- NT318 pad 1: Net-(IC302-CTRC) -> Net-(IC302-CTRD)
- NT334 pad 2: Net-(C329-Pad1) -> Net-(NT334-Pad2)
- NT335 pad 2: Net-(C329-Pad1) -> Net-(NT334-Pad2)
- Q309 pad 3: Net-(C329-Pad1) -> Net-(NT334-Pad2)
- R329 pad 1: Net-(NT319-Pad1) -> Net-(NT317-Pad1)
- R331 pad 1: Net-(NT320-Pad1) -> Net-(NT317-Pad1)
- R334 pad 1: Net-(NT322-Pad1) -> Net-(Q310-S)
- R340 pad 1: Net-(NT325-Pad1) -> Net-(Q305-S)
- R344 pad 1: Net-(NT329-Pad1) -> Net-(Q306-S)
- R350 pad 2: Net-(C329-Pad1) -> Net-(NT334-Pad2)
- TPe213 pad 1: USB_C_GPIO -> Net-(U202-GPIO_1)
- U202 pad 25: (no net) -> PACK -
- U202 pad 8: USB_C_GPIO -> Net-(U202-GPIO_1)
- U401 pad 15: (no net) -> unconnected-(U401-TP-Pad15)
- U401 pad 7: Net-(U401-Pad7) -> unconnected-(U401-Pad7)
- U401 pad 9: Net-(U401-Pad7) -> unconnected-(U401-Pad9)
Routing:
- net Net-(Q306-S): track 7.76 -> 192.8 mm, vias 0 -> 5
- net Net-(Q310-S): track 9.59 -> 131.5 mm, vias 0 -> 3
- net /uc_stage/digLED1_Red_EN: track 0.00 -> 104.4 mm, vias 0 -> 2
- net /uc_stage/digLED2_Orange_EN: track 0.00 -> 100.8 mm, vias 0 -> 2
- net /uc_stage/digLED3_Green_EN: track 0.00 -> 96.5 mm, vias 0 -> 2
- net /uc_stage/digLED4_Green_EN: track 0.00 -> 91.0 mm, vias 0 -> 2
- net digCharge_EN: track 0.00 -> 64.3 mm, vias 0 -> 2
- net EXT_5V: track 0.00 -> 60.2 mm, vias 0 -> 2
- net Net-(Q302-G): track 4.12 -> 63.7 mm, vias 0 -> 4
- net HPI_SCL: track 7.63 -> 66.7 mm, vias 0 -> 2
- net HPI_SDA: track 9.24 -> 67.5 mm, vias 0 -> 2
- net Net-(Q304A-E1): track 0.00 -> 54.2 mm, vias 0 -> 2
- net anUSBVoltage: track 6.81 -> 57.8 mm, vias 0 -> 2
- net /uc_stage/SW_5V: track 0.00 -> 49.7 mm, vias 0 -> 4
- net VREG_3V3: track 12.5 -> 55.3 mm, vias 0 -> 7
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- added copper zone on In2.Cu, net /battery_management/BAT23
- added copper zone on F.Cu, net Earth
- added copper zone on In1.Cu, net Earth
- added copper zone on B.Cu, net Net-(L301-Pad1)
- added copper zone on F.Cu, net Net-(L301-Pad1)
- added copper zone on In2.Cu, net Net-(L301-Pad1)
- added copper zone on F.Cu, net Net-(L301-Pad2)
- added copper zone on In2.Cu, net Net-(L301-Pad2)
- added copper zone on F.Cu, net Net-(NT334-Pad2)
- added copper zone on In2.Cu, net Net-(NT334-Pad2)
- added copper zone on F.Cu, net Net-(Q309-Pad5)
- added copper zone on In2.Cu, net Net-(Q309-Pad5)
- added copper zone on F.Cu, net PACK +
- added copper zone on In2.Cu, net PACK +
- added copper zone on B.Cu, net USB_C_BUS
- added copper zone on In2.Cu, net VREG_3V3
- added copper zone on F.Cu, net V_SYSTEM
- added copper zone on In2.Cu, net V_SYSTEM
